File: _Cap Sense Core Tech/CapSense/Hardware/CapSenseDuo/_autosave-CapSenseDuo.kicad_sch (KiCad schematic)
At the start: 39 parts, among them IC1 FDC2214-rescue_FDC2214QRGHRQ1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, IC2 FDC2214QRGHRQ1, J1 Conn_01x08, J2 Conn_01x08, Y1 ECS-2033-400-BN

Commit message: layout pre route
Parts:
- gave numbers to parts that had none: 1
Changed lines of the file:
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@@
   (symbol (lib_id "Switch:SW_Push_DPDT") (at 80.01 168.91 0) (unit 1)
     (in_bom yes) (on_board yes) (fields_autoplaced)
-    (property "Reference" "SW?" (id 0) (at 80.01 156.21 0))
+    (property "Reference" "SW1" (id 0) (at 80.01 156.21 0))
     (property "Value" "SW_Push_DPDT" (id 1) (at 80.01 158.75 0))
     (property "Footprint" "SamacSys:2mm-DPDT" (id 2) (at 80.01 163.83 0)
@@
     )
     (path "/33a21ba8-7858-449f-82f5-cbfa2271ef38"
-      (reference "SW?") (unit 1) (value "SW_Push_DPDT") (footprint "SamacSys:2mm-DPDT")
+      (reference "SW1") (unit 1) (value "SW_Push_DPDT") (footprint "SamacSys:2mm-DPDT")
     )
     (path "/00000000-0000-0000-0000-000060da4d63"
