File: _Cap Sense Core Tech/CapSense/Hardware/CapSenseDuo 2/CapSenseDuo.kicad_pcb (KiCad board)
At the start: 2 copper layers, 30 x 51.3 mm, 48 parts, among them IC1 FDC2214-rescue_FDC2214QRGHRQ1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, IC2 FDC2214QRGHRQ1, J1 Conn_02x04_Odd_Even, J2 Conn_02x04_Odd_Even, J3 Conn_02x01, SW1 SW_Push_DPDT, Y1 ECS-2033-400-BN

Commit message: pcb
Changed lines of the file:
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@@
       (outputformat 1)
       (mirror false)
-      (drillshape 0)
+      (drillshape 1)
       (scaleselection 1)
-      (outputdirectory "Output")
+      (outputdirectory "")
     )
   )
@@
     (pad "17" smd rect locked (at 0 -0.000003 315) (size 2.6 2.6) (layers "F.Cu" "F.Mask")
       (net 1 "GND") (pinfunction "DAP") (pintype "passive"))
-    (pad "V" smd circle locked (at 0 1.05 315) (size 0.499999 0.499999) (layers "F.Cu" "F.Paste" "F.Mask")
+    (pad "V" thru_hole circle locked (at 0 1.05 315) (size 0.499999 0.499999) (drill 0.2032) (layers *.Cu *.Mask)
       (net 1 "GND"))
-    (pad "V" smd circle locked (at 0 -1.05 315) (size 0.499999 0.499999) (layers "F.Cu" "F.Paste" "F.Mask")
+    (pad "V" thru_hole circle locked (at 0 -1.05 315) (size 0.499999 0.499999) (drill 0.2032) (layers *.Cu *.Mask)
       (net 1 "GND"))
-    (pad "V" thru_hole circle locked (at 0 -0.000003 315) (size 2.5 2.5) (drill 2) (layers *.Cu *.Mask)
+    (pad "V" thru_hole circle locked (at 0 -0.000003 315) (size 0.499999 0.499999) (drill 0.2032) (layers *.Cu *.Mask)
       (net 1 "GND"))
-    (pad "V" smd circle locked (at -1.05 -0.000003 315) (size 0.499999 0.499999) (layers "F.Cu" "F.Paste" "F.Mask")
+    (pad "V" thru_hole circle locked (at -1.05 -0.000003 315) (size 0.499999 0.499999) (drill 0.2032) (layers *.Cu *.Mask)
       (net 1 "GND"))
-    (pad "V" smd circle locked (at 1.05 -0.000003 315) (size 0.499999 0.499999) (layers "F.Cu" "F.Paste" "F.Mask")
+    (pad "V" thru_hole circle locked (at 1.05 -0.000003 315) (size 0.499999 0.499999) (drill 0.2032) (layers *.Cu *.Mask)
       (net 1 "GND"))
     (model "/Users/zhoubo/Documents/KiCad/6.0/3dmodels/FDC2214QRGHRQ1.stp"
@@
     (pad "17" smd rect locked (at 0 -0.000003 315) (size 2.6 2.6) (layers "F.Cu" "F.Mask")
       (net 1 "GND") (pinfunction "DAP") (pintype "passive"))
-    (pad "V" smd circle locked (at 0 -1.05 315) (size 0.499999 0.499999) (layers "F.Cu" "F.Paste" "F.Mask")
+    (pad "V" thru_hole circle locked (at 0 -1.05 315) (size 0.499999 0.499999) (drill 0.2032) (layers *.Cu *.Mask)
       (net 1 "GND"))
-    (pad "V" thru_hole circle locked (at 0 -0.000003 315) (size 2.4 2.4) (drill 2) (layers *.Cu *.Mask)
+    (pad "V" thru_hole circle locked (at 0 -0.000003 315) (size 0.499999 0.499999) (drill 0.2032) (layers *.Cu *.Mask)
       (net 1 "GND"))
-    (pad "V" smd circle locked (at -1.05 -0.000003 315) (size 0.499999 0.499999) (layers "F.Cu" "F.Paste" "F.Mask")
+    (pad "V" thru_hole circle locked (at -1.05 -0.000003 315) (size 0.499999 0.499999) (drill 0.2032) (layers *.Cu *.Mask)
       (net 1 "GND"))
-    (pad "V" smd circle locked (at 0 1.05 315) (size 0.499999 0.499999) (layers "F.Cu" "F.Paste" "F.Mask")
+    (pad "V" thru_hole circle locked (at 0 1.05 315) (size 0.499999 0.499999) (drill 0.2032) (layers *.Cu *.Mask)
       (net 1 "GND"))
-    (pad "V" smd circle locked (at 1.05 -0.000003 315) (size 0.499999 0.499999) (layers "F.Cu" "F.Paste" "F.Mask")
+    (pad "V" thru_hole circle locked (at 1.05 -0.000003 315) (size 0.499999 0.499999) (drill 0.2032) (layers *.Cu *.Mask)
       (net 1 "GND"))
     (model "/Users/zhoubo/Documents/KiCad/6.0/3dmodels/FDC2214QRGHRQ1.stp"
@@
   (segment (start 111.760002 114.72566) (end 111.760002 114.239508) (width 0.25) (layer "F.Cu") (net 1))
   (segment (start 110.063629 113.664998) (end 108.712 113.664998) (width 0.25) (layer "F.Cu") (net 1))
+  (segment (start 111.760002 113.664998) (end 111.760002 109.728002) (width 0.25) (layer "F.Cu") (net 1))
   (segment (start 110.946829 139.673999) (end 111.760002 138.860826) (width 0.25) (layer "F.Cu") (net 1))
   (segment (start 111.760002 138.860826) (end 111.760002 138.374674) (width 0.25) (layer "F.Cu") (net 1))
@@
   (segment (start 111.760002 134.112002) (end 111.76 134.112) (width 0.25) (layer "F.Cu") (net 1))
   (segment (start 105.3865 136.652) (end 105.3865 138.1215) (width 0.25) (layer "F.Cu") (net 1))
-  (segment (start 111.76 113.665) (end 111.760002 113.664998) (width 0.25) (layer "F.Cu") (net 1))
-  (segment (start 111.760002 113.664998) (end 111.760002 109.728002) (width 0.25) (layer "F.Cu") (net 1))
   (segment (start 110.6932 140.7792) (end 111.519 141.605) (width 0.25) (layer "F.Cu") (net 1))
   (via (at 111.646 118.986) (size 0.8) (drill 0.4) (layers "F.Cu" "B.Cu") (net 1))
