File: _Cap Sense Core Tech/CapSense/Hardware/CapSenseQuadro/CapSenseQuadro.kicad_sch (KiCad schematic)
At the start: 48 parts, among them IC1 FDC2214-rescue_FDC2214QRGHRQ1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, IC2 FDC2214QRGHRQ1, J1 Conn_02x04_Odd_Even, J2 Conn_02x04_Odd_Even, J3 Conn_02x01, SW1 SW_Push_DPDT, Y1 ECS-2033-400-BN

Commit message: pcb
Parts:
- removed J1, J2: Conn_02x04_Odd_Even, Connector_PinHeader_2.54mm:PinHeader_2x04_P2.54mm_Horizontal, symbol Connector_Generic:Conn_02x04_Odd_Even
- removed R10, R11: R, Resistor_SMD:R_0603_1608Metric_Pad0.98x0.95mm_HandSolder, symbol Device:R
- added C16, C17, C18, C23, C24, C25: C, Capacitor_SMD:C_0603_1608Metric, symbol Device:C
- added C19, C20, C21, C22, C26, C27, C28, C29: Device_C, Capacitor_SMD:C_0603_1608Metric, symbol FDC2214:Device_C
- added IC3, IC4: FDC2214QRGHRQ1, FDC2214:FDC2214RGHR, symbol FDC2214:FDC2214-rescue_FDC2214QRGHRQ1-SamacSys_Parts
- added IC5: PCA9543APWR, SOP65P640X120-14N, symbol SamacSys:PCA9543APWR
- added J1, J2: Conn_02x08_Odd_Even, Connector_PinHeader_2.54mm:PinHeader_2x08_P2.54mm_Horizontal, symbol Connector_Generic:Conn_02x08_Odd_Even
- added L10, L11, L12, L13, L14, L15, L16, L9: L0806C470MPWST, INDC2018X180N, symbol SamacSys:L0806C470MPWST
- added R12, R13, R14, R15, R16, R17, R20, R21, R22: R, Resistor_SMD:R_0603_1608Metric_Pad0.98x0.95mm_HandSolder, symbol Device:R
Connections:
- net +3V3: now also C16.1, C17.1, C18.1, C23.1, C24.1, C25.1, IC3.7 (VDD), IC4.7 (VDD), IC5.14 (VCC), R12.1, R14.1, R16.2, R17.1
- net ADDR1: no longer A1.19 (D0)
- net ADDR2: no longer A1.20 (D1)
- net GND: now also C16.2, C17.2, C18.2, C23.2, C24.2, C25.2, IC3.17 (DAP), IC3.8 (GND), IC4.17 (DAP), IC4.8 (GND), IC5.7 (GND), R13.2, R15.2, R20.2, R21.2, R22.2
- net IN0A: now also J1.1 (Pin_1)
- net IN0B: now also J1.2 (Pin_2)
- net IN1A: now also J1.3 (Pin_3)
- net IN1B: now also J1.4 (Pin_4)
- net IN2A: now also J1.5 (Pin_5)
- net IN2B: now also J1.6 (Pin_6)
- net IN3A: now also J1.7 (Pin_7)
- net IN3B: now also J1.8 (Pin_8)
- net IN4A: now also J1.9 (Pin_9)
- net IN4B: now also J1.10 (Pin_10)
- net IN5A: now also J1.11 (Pin_11)
- net IN5B: now also J1.12 (Pin_12)
- net IN6A: now also J1.13 (Pin_13)
- net IN6B: now also J1.14 (Pin_14)
- net IN7A: now also J1.15 (Pin_15)
- net IN7B: now also J1.16 (Pin_16)
- net INTB2: now also IC3.5 (INTB), IC4.5 (INTB)
- net SCL: now also IC5.12 (SCL); no longer IC1.1 (SCL), R4.2
- net SDA: now also IC5.13 (SDA); no longer IC1.2 (SDA), R3.2
- net clk: now also IC3.3 (CLKIN), IC4.3 (CLKIN)
- net SCL2 renamed SCL0
- net SCL0: now also IC1.1 (SCL), R4.2, IC5.6 (SC0)
- net SD renamed SD1
- net SD1: no longer A1.21 (D2), IC2.6 (SD)
- net SDA2 renamed SDA0
- net SDA0: now also IC1.2 (SDA), R3.2, IC5.5 (SD0)
- new net ADDR3: IC3.4 (ADDR), R12.2, R13.1
- new net ADDR4: IC4.4 (ADDR), R14.2, R15.1
- new net IN10A: C20.2, IC3.13 (IN2A), J2.5 (Pin_5), L10.1
- new net IN10B: C20.1, IC3.14 (IN2B), J2.6 (Pin_6), L10.2
- new net IN11A: C19.2, IC3.15 (IN3A), J2.7 (Pin_7), L9.1
- new net IN11B: C19.1, IC3.16 (IN3B), J2.8 (Pin_8), L9.2
- new net IN12A: C29.2, IC4.9 (IN0A), J2.9 (Pin_9), L16.1
- new net IN12B: C29.1, IC4.10 (IN0B), J2.10 (Pin_10), L16.2
- new net IN13A: C28.2, IC4.11 (IN1A), J2.11 (Pin_11), L15.1
- new net IN13B: C28.1, IC4.12 (IN1B), J2.12 (Pin_12), L15.2
- new net IN14A: C27.2, IC4.13 (IN2A), J2.13 (Pin_13), L14.1
- new net IN14B: C27.1, IC4.14 (IN2B), J2.14 (Pin_14), L14.2
- new net IN15A: C26.2, IC4.15 (IN3A), J2.15 (Pin_15), L13.1
- new net IN15B: C26.1, IC4.16 (IN3B), J2.16 (Pin_16), L13.2
- new net IN8A: C22.2, IC3.9 (IN0A), J2.1 (Pin_1), L12.1
- new net IN8B: C22.1, IC3.10 (IN0B), J2.2 (Pin_2), L12.2
- new net IN9A: C21.2, IC3.11 (IN1A), J2.3 (Pin_3), L11.1
- new net IN9B: C21.1, IC3.12 (IN1B), J2.4 (Pin_4), L11.2
- new net PCA0: A1.19 (D0), IC5.1 (A0)
- new net PCA1: A1.20 (D1), IC5.2 (A1)
- new net SCL1: IC3.1 (SCL), IC4.1 (SCL), IC5.10 (SC1), R17.2
- new net SD2: IC2.6 (SD), R21.1
- new net SD3: IC3.6 (SD), R20.1
- new net SD4: IC4.6 (SD), R22.1
- new net SDA1: IC3.2 (SDA), IC4.2 (SDA), IC5.9 (SD1), R16.1
Other:
- moved on the sheet: C10, C11, C12, C13, C14, C15, C9, IC2, J3, L5, L6, L7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
